File: pcb/macropad.kicad_sch (KiCad schematic)
At the start: 14 parts, among them SW1 SW_Push, SW10 RotaryEncoder_Switch, SW2 SW_Push, SW3 SW_Push, SW4 SW_Push, SW5 SW_Push, SW6 SW_Push, SW7 SW_Push, SW8 SW_Push, SW9 SW_Push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

Commit message: added more pcb files
Connections:
- net row0 renamed row is col 0
Changed lines of the file:
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@@
 		)
 	)
-	(label "row0"
+	(label "row is col 0"
 		(at 83.82 81.28 0)
 		(effects
